File: alim/_saved_protodual.sch (KiCad schematic (older format))
At the start: 61 parts, among them P1 BAT1+, P2 BAT1-, P3 ALIM_PW1, P4 ARU, P5 BAT2+, P6 BAT2-, Q1 Q_NMOS_DGS, Q2 Q_NMOS_DGS, Q3 Q_NMOS_DGS, Q4 Q_NMOS_DGS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

Commit message: ALim a grosse piste
Parts:
- R11: value 3M1W -> 3m1W
- R6: value 5M1.5W -> 5m1.5W
Connections:
- net FBCK1: now also U1.16 (FB2); no longer U1.9 (FB1)
- net FBCK2: now also U1.9 (FB1); no longer U1.16 (FB2)
- net at C10.1, D1.2 (A): now also U1.24 (VCC2); no longer U1.1 (VCC1)
- net at C6.2, R4.2: now also U1.15 (COMP2); no longer U1.10 (COMP1)
- net at U1.2 (LO1): now also Q4.2 (G); no longer Q2.2 (G)
- net at C11.2, D1.1 (K): now also U1.27 (HB2); no longer U1.30 (HB1)
- net at U1.31 (HO1): now also Q3.2 (G); no longer Q1.2 (G)
- net at C11.1, L1.1, Q1.3 (S)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: now also U1.25 (SW2); no longer U1.32 (SW1)
- net at Q2.3 (S), R6.1: now also U1.20 (CS2); no longer U1.5 (CS1)
- net at C7.1, R5.2: now also U1.19 (RAMP2); no longer U1.6 (RAMP1)
- net at U1.7 (SS1): now also C15.1; no longer C9.1
- net at C12.2, R7.2: now also U1.10 (COMP1); no longer U1.15 (COMP2)
- net at U1.18 (SS2): now also C9.1; no longer C15.1
- net at C13.1, R10.1: now also U1.6 (RAMP1); no longer U1.19 (RAMP2)
- net at Q4.3 (S), R11.1: now also U1.5 (CS1); no longer U1.20 (CS2)
- net at U1.23 (LO2): now also Q2.2 (G); no longer Q4.2 (G)
- net at C23.1, D2.2 (A): now also U1.1 (VCC1); no longer U1.24 (VCC2)
- net at C31.2, L2.1, Q3.3 (S)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: now also U1.32 (SW1); no longer U1.25 (SW2)
- net at U1.26 (HO2): now also Q1.2 (G); no longer Q3.2 (G)
- net at C31.1, D2.1 (K): now also U1.30 (HB1); no longer U1.27 (HB2)
Other:
- moved on the sheet: U1A, U1B
Changed lines of the file:
@@
 L LM25119 U1
 U 1 1 5A2F183E
-P 5950 4050
-F 0 "U1" H 5850 4650 50  0000 R CNN
-F 1 "LM25119" H 5850 4550 50  0000 R CNN
-F 2 "Housings_DFN_QFN:QFN-32-1EP_5x5mm_Pitch0.5mm" H 5950 4050 50  0001 C CNN
-F 3 "" H 5950 4050 50  0001 C CNN
-	1    5950 4050
+P 8700 4050
+F 0 "U1" H 8600 4650 50  0000 R CNN
+F 1 "LM25119" H 8600 4550 50  0000 R CNN
+F 2 "Housings_DFN_QFN:QFN-32-1EP_5x5mm_Pitch0.5mm" H 8700 4050 50  0001 C CNN
+F 3 "" H 8700 4050 50  0001 C CNN
+	1    8700 4050
 	1    0    0    -1
 $EndComp
@@
 L LM25119 U1
 U 2 1 5A2F1A68
-P 8700 4050
-F 0 "U1" H 8600 4650 50  0000 R CNN
-F 1 "LM25119" H 8600 4550 50  0000 R CNN
-F 2 "Housings_DFN_QFN:QFN-32-1EP_5x5mm_Pitch0.5mm" H 8700 4050 50  0001 C CNN
-F 3 "" H 8700 4050 50  0001 C CNN
-	2    8700 4050
+P 5950 4050
+F 0 "U1" H 5850 4650 50  0000 R CNN
+F 1 "LM25119" H 5850 4550 50  0000 R CNN
+F 2 "Housings_DFN_QFN:QFN-32-1EP_5x5mm_Pitch0.5mm" H 5950 4050 50  0001 C CNN
+F 3 "" H 5950 4050 50  0001 C CNN
+	2    5950 4050
 	1    0    0    -1
 $EndComp
@@
 	1    0    0    -1
 $EndComp
-NoConn ~ 8100 4250
+NoConn ~ 5350 4250
 $Comp
 L C_Small C8
@@
 P 7400 3050
 F 0 "R6" H 7430 3070 50  0000 L CNN
-F 1 "5M1.5W" H 7430 3010 50  0000 L CNN
+F 1 "5m1.5W" H 7430 3010 50  0000 L CNN
 F 2 "Resistors_SMD:R_2010_HandSoldering" H 7400 3050 50  0001 C CNN
 F 3 "" H 7400 3050 50  0001 C CNN
@@
 P 10150 3050
 F 0 "R11" H 10180 3070 50  0000 L CNN
-F 1 "3M1W" H 10180 3010 50  0000 L CNN
+F 1 "3m1W" H 10180 3010 50  0000 L CNN
 F 2 "Resistors_SMD:R_2010_HandSoldering" H 10150 3050 50  0001 C CNN
 F 3 "" H 10150 3050 50  0001 C CNN
