File: alim/protodual.sch (KiCad schematic (older format))
At the start: 56 parts, among them Q1 Q_NMOS_DGS, Q2 Q_NMOS_DGS, Q3 Q_NMOS_DGS, Q4 Q_NMOS_DGS, U1 LM25119

Commit message: Proto dual
Parts:
- added P1: CONN_01X02, kicad-library:BATT_SOLDERPAD, symbol CONN_01X02
- added P2, P3: CONN_01X02, Connectors_Molex:Molex_MiniFit-JR-5556-02A_2x01x4.20mm_Straight, symbol CONN_01X02
- C10, C11, C12, C13, C14, C23, C31, C4, C6, C7, C8: footprint Capacitors_SMD:C_0402 -> Capacitors_SMD:C_0603_HandSoldering
- Q1, Q2, Q3, Q4: footprint (none) -> kicad-library:TDSON8_MOSFET
- R1, R10, R12, R13, R2, R3, R4, R5, R7, R8, R9: footprint (none) -> Resistors_SMD:R_0603_HandSoldering
- R11, R6: footprint (none) -> Resistors_SMD:R_2010_HandSoldering
- U1: footprint (none) -> Housings_DFN_QFN:QFN-32-1EP_5x5mm_Pitch0.5mm
Connections:
- net +BATT: now also P1.2 (P2)
- net GND: now also P1.1 (P1), P2.1 (P1), P3.1 (P1)
- net VOUT1: now reaches C16.1, C17.1, C18.1, C19.1, C20.1, C21.1, C22.1, C24.1, C25.1, C26.1, C27.1, C28.1, C29.1, C30.1, L1.2, R8.1
- net VOUT1: now also P2.2 (P2)
- net VOUT2: now reaches C32.1, C33.1, C34.1, L2.2, R12.1
- net VOUT2: now also P3.2 (P2)

Commit message: MAJ alim + couleur
Parts:
- removed P2, P3: CONN_01X02, Connectors_Molex:Molex_MiniFit-JR-5556-02A_2x01x4.20mm_Straight, symbol CONN_01X02
- added C35, C36, C37: 22uF/50V, Capacitors_SMD:C_1206_HandSoldering, symbol C_Small
- added F1: 15A, Fuse_Holders_and_Fuses:Fuseholder5x20_horiz_SemiClosed_Casing10x25mm, symbol Fuse_Small
- added P2: ALIM_L1, Pin_Headers:Pin_Header_Straight_2x03, symbol CONN_02X03
- added P3: ALIM_PW1, Pin_Headers:Pin_Header_Straight_2x16, symbol CONN_02X16
- added P4: ARU, Socket_Strips:Socket_Strip_Straight_1x02, symbol CONN_01X02
- added P5: SW_LOGIC, Socket_Strips:Socket_Strip_Straight_1x02, symbol CONN_01X02
- added Q5, Q6: Q_PMOS_GDS, TO_SOT_Packages_SMD:SOT-428, symbol Q_PMOS_GDS
- added R14, R15: 10k, Resistors_SMD:R_0603_HandSoldering, symbol R_Small
- added U2: TRACO3.3, kicad-library:TRACO-TSR-1-DC-DC, symbol 7805-RESCUE-Alimentation_2017
- added U3: TRACO5, kicad-library:TRACO-TSR-1-DC-DC, symbol 7805-RESCUE-Alimentation_2017
- added U4: TRACO15, kicad-library:TRACO-TSR-1-DC-DC, symbol 7805-RESCUE-Alimentation_2017
- P1: value CONN_01X02 -> BATT_IN
Connections:
- net +BATT: now also P3.10 (P10), P3.2 (P2), P3.4 (P4), P3.6 (P6), P3.8 (P8), P4.1 (P1), Q5.3 (S); no longer P1.2 (P2)
- net GND: now also U1.33 (EP), C35.2, C36.2, C37.2, P2.4 (P4), P2.5 (P5), P2.6 (P6), P3.12 (P12), P3.14 (P14), P3.16 (P16), P3.18 (P18), P3.20 (P20), P3.22 (P22), P3.24 (P24), P3.26 (P26), P3.28 (P28), P3.29 (P29), P3.30 (P30), P3.31 (P31), P3.32 (P32), U2.GND, U3.GND, U4.GND
- net VOUT1: now also P3.15 (P15), P3.17 (P17), P3.19 (P19), P3.21 (P21), P3.23 (P23), P3.25 (P25), P3.27 (P27)
- net VOUT2: now also P3.1 (P1), P3.11 (P11), P3.13 (P13), P3.3 (P3), P3.5 (P5), P3.7 (P7), P3.9 (P9)
- new net: F1.1, P1.2 (P2)
- new net: C35.1, C36.1, C37.1, P5.1 (P1), Q6.3 (S), U2.VI, U3.VI, U4.VI
- new net: P4.2 (P2), Q5.1 (G), R14.2
- new net: P5.2 (P2), Q6.1 (G), R15.2
- new net VBATT: F1.2, Q5.2 (D), Q6.2 (D), R14.1, R15.1
- new net VL15: P2.3 (P3), U4.VO
- new net VL33: P2.1 (P1), U2.VO
- new net VL5: P2.2 (P2), U3.VO
Other:
- moved on the sheet: P1

Commit message: Alim finale?
Parts:
- added R16, R17: 1k, Resistors_SMD:R_0603_HandSoldering, symbol R_Small
- R14, R15: value 10k -> 20k
Connections:
- net +BATT: no longer P4.1 (P1)
- net GND: now also P4.1 (P1), P5.1 (P1)
- net at C35.1, C36.1, C37.1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: no longer P5.1 (P1)
- net at Q5.1 (G), R14.2: now also R16.1; no longer P4.2 (P2)
- net at Q6.1 (G), R15.2: now also R17.2; no longer P5.2 (P2)
- new net: P4.2 (P2), R16.2
- new net: P5.2 (P2), R17.1
Changed lines of the file:
@@
 L +BATT #PWR013
 U 1 1 5A63CB75
-P 1850 2100
-F 0 "#PWR013" H 1850 1950 50  0001 C CNN
-F 1 "+BATT" H 1850 2240 50  0000 C CNN
-F 2 "" H 1850 2100 50  0001 C CNN
-F 3 "" H 1850 2100 50  0001 C CNN
-	1    1850 2100
+P 1950 2100
+F 0 "#PWR013" H 1950 1950 50  0001 C CNN
+F 1 "+BATT" H 1950 2240 50  0000 C CNN
+F 2 "" H 1950 2100 50  0001 C CNN
+F 3 "" H 1950 2100 50  0001 C CNN
+	1    1950 2100
 	-1   0    0    1
 $EndComp
@@
 $EndComp
 Wire Wire Line
-	1300 5850 4050 5850
-Wire Wire Line
 	3050 5850 3050 6200
 Connection ~ 2000 5850
@@
 P 1550 1500
 F 0 "R14" H 1580 1520 50  0000 L CNN
-F 1 "10k" H 1580 1460 50  0000 L CNN
+F 1 "20k" H 1580 1460 50  0000 L CNN
 F 2 "Resistors_SMD:R_0603_HandSoldering" H 1550 1500 50  0001 C CNN
 F 3 "" H 1550 1500 50  0001 C CNN
@@
 	1550 1400 1550 1250
 Connection ~ 1550 1250
-Wire Wire Line
-	1550 1900 1200 1900
 Connection ~ 1550 1750
-Wire Wire Line
-	1200 2000 1950 2000
-Connection ~ 1850 2000
-Wire Wire Line
-	1700 5750 1300 5750
 Wire Wire Line
 	1700 5400 1700 5750
@@
 P 1700 5300
 F 0 "R15" H 1730 5320 50  0000 L CNN
-F 1 "10k" H 1730 5260 50  0000 L CNN
+F 1 "20k" H 1730 5260 50  0000 L CNN
 F 2 "Resistors_SMD:R_0603_HandSoldering" H 1700 5300 50  0001 C CNN
 F 3 "" H 1700 5300 50  0001 C CNN
@@
 	1650 1750 1550 1750
 Wire Wire Line
-	1950 2000 1950 1950
-Wire Wire Line
-	1850 2000 1850 2100
+	1950 2100 1950 1950
 $Comp
 L Q_PMOS_GDS Q6
@@
 	3550 4650 3550 4900
 Connection ~ 3550 4900
+$Comp
+L GND #PWR019
+U 1 1 5A7F2961
+P 1550 2000
+F 0 "#PWR019" H 1550 1750 50  0001 C CNN
+F 1 "GND" H 1550 1850 50  0000 C CNN
+F 2 "" H 1550 2000 50  0001 C CNN
+F 3 "" H 1550 2000 50  0001 C CNN
+	1    1550 2000
+	1    0    0    -1
+$EndComp
+Wire Wire Line
+	1200 2000 1550 2000
+$Comp
+L R_Small R16
+U 1 1 5A7F3154
+P 1350 1900
+F 0 "R16" V 1250 1850 50  0000 L CNN
+F 1 "1k" V 1350 1850 50  0000 L CNN
+F 2 "Resistors_SMD:R_0603_HandSoldering" H 1350 1900 50  0001 C CNN
+F 3 "" H 1350 1900 50  0001 C CNN
+	1    1350 1900
+	0    1    1    0
+$EndComp
+Wire Wire Line
+	1550 1900 1450 1900
+Wire Wire Line
+	1200 1900 1250 1900
+Wire Wire Line
+	2000 5850 4050 5850
+$Comp
+L R_Small R17
+U 1 1 5A7F4B3D
+P 1500 5750
+F 0 "R17" H 1530 5770 50  0000 L CNN
+F 1 "1k" H 1530 5710 50  0000 L CNN
+F 2 "Resistors_SMD:R_0603_HandSoldering" H 1500 5750 50  0001 C CNN
+F 3 "" H 1500 5750 50  0001 C CNN
+	1    1500 5750
+	0    -1   -1   0
+$EndComp
+Wire Wire Line
+	1300 5750 1400 5750
+Wire Wire Line
+	1700 5750 1600 5750
+$Comp
+L GND #PWR020
+U 1 1 5A7F520B
+P 1700 5850
+F 0 "#PWR020" H 1700 5600 50  0001 C CNN
+F 1 "GND" H 1700 5700 50  0000 C CNN
+F 2 "" H 1700 5850 50  0001 C CNN
+F 3 "" H 1700 5850 50  0001 C CNN
+	1    1700 5850
+	1    0    0    -1
+$EndComp
+Wire Wire Line
+	1300 5850 1700 5850
 $EndSCHEMATC

Commit message: Alim
Parts:
- removed C35, C36, C37: 22uF/50V, Capacitors_SMD:C_1206_HandSoldering, symbol C_Small
- added C35, C36, C37: 22uF/50V, Capacitors_SMD:c_elec_6.3x5.3, symbol CP1_Small
- D1, D2: footprint Diodes_SMD:SMC_Handsoldering -> Diodes_SMD:D_0805
- R14, R15: value 20k -> 10k
- R16, R17: value 1k -> 8k
Connections:
- net GND: now also C35.2, C36.2, C37.2
- net at Q6.3 (S), U2.VI, U3.VI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: now also C35.1, C36.1, C37.1
Changed lines of the file:
@@
 F 0 "D1" H 6200 3550 50  0000 C CNN
 F 1 "500mV@50V" H 6200 3350 50  0000 C CNN
-F 2 "Diodes_SMD:SMC_Handsoldering" H 6200 3450 50  0001 C CNN
+F 2 "Diodes_SMD:D_0805" H 6200 3450 50  0001 C CNN
 F 3 "" H 6200 3450 50  0001 C CNN
 	1    6200 3450
@@
 F 0 "D2" H 8950 3550 50  0000 C CNN
 F 1 "500mV@50V" H 8950 3350 50  0000 C CNN
-F 2 "Diodes_SMD:SMC_Handsoldering" H 8950 3450 50  0001 C CNN
+F 2 "Diodes_SMD:D_0805" H 8950 3450 50  0001 C CNN
 F 3 "" H 8950 3450 50  0001 C CNN
 	1    8950 3450
@@
 	4450 6500 4450 6400
 Connection ~ 3450 6500
-$Comp
-L C_Small C35
-U 1 1 5A6714FD
-P 2000 6300
-F 0 "C35" H 2010 6370 50  0000 L CNN
-F 1 "22uF/50V" H 2010 6220 50  0000 L CNN
-F 2 "Capacitors_SMD:C_1206_HandSoldering" H 2000 6300 50  0001 C CNN
-F 3 "" H 2000 6300 50  0001 C CNN
-	1    2000 6300
-	1    0    0    -1
-$EndComp
 Connection ~ 2000 6100
 Connection ~ 2000 6500
-$Comp
-L C_Small C36
-U 1 1 5A671A87
-P 3050 6300
-F 0 "C36" H 3060 6370 50  0000 L CNN
-F 1 "22uF/50V" H 3060 6220 50  0000 L CNN
-F 2 "Capacitors_SMD:C_1206_HandSoldering" H 3050 6300 50  0001 C CNN
-F 3 "" H 3050 6300 50  0001 C CNN
-	1    3050 6300
-	1    0    0    -1
-$EndComp
 Connection ~ 3050 6100
 Wire Wire Line
 	3050 6400 3050 6500
 Connection ~ 3050 6500
-$Comp
-L C_Small C37
-U 1 1 5A671F3A
-P 4050 6300
-F 0 "C37" H 4060 6370 50  0000 L CNN
-F 1 "22uF/50V" H 4060 6220 50  0000 L CNN
-F 2 "Capacitors_SMD:C_1206_HandSoldering" H 4050 6300 50  0001 C CNN
-F 3 "" H 4050 6300 50  0001 C CNN
-	1    4050 6300
-	1    0    0    -1
-$EndComp
 Connection ~ 4050 6100
 Wire Wire Line
@@
 P 1550 1500
 F 0 "R14" H 1580 1520 50  0000 L CNN
-F 1 "20k" H 1580 1460 50  0000 L CNN
+F 1 "10k" H 1580 1460 50  0000 L CNN
 F 2 "Resistors_SMD:R_0603_HandSoldering" H 1550 1500 50  0001 C CNN
 F 3 "" H 1550 1500 50  0001 C CNN
@@
 P 1700 5300
 F 0 "R15" H 1730 5320 50  0000 L CNN
-F 1 "20k" H 1730 5260 50  0000 L CNN
+F 1 "10k" H 1730 5260 50  0000 L CNN
 F 2 "Resistors_SMD:R_0603_HandSoldering" H 1700 5300 50  0001 C CNN
 F 3 "" H 1700 5300 50  0001 C CNN
@@
 P 1350 1900
 F 0 "R16" V 1250 1850 50  0000 L CNN
-F 1 "1k" V 1350 1850 50  0000 L CNN
+F 1 "8k" V 1350 1850 50  0000 L CNN
 F 2 "Resistors_SMD:R_0603_HandSoldering" H 1350 1900 50  0001 C CNN
 F 3 "" H 1350 1900 50  0001 C CNN
@@
 P 1500 5750
 F 0 "R17" H 1530 5770 50  0000 L CNN
-F 1 "1k" H 1530 5710 50  0000 L CNN
+F 1 "8k" H 1530 5710 50  0000 L CNN
 F 2 "Resistors_SMD:R_0603_HandSoldering" H 1500 5750 50  0001 C CNN
 F 3 "" H 1500 5750 50  0001 C CNN
@@
 Wire Wire Line
 	1300 5850 1700 5850
+$Comp
+L CP1_Small C35
+U 1 1 5A835D32
+P 2000 6300
+F 0 "C35" H 2010 6370 50  0000 L CNN
+F 1 "22uF/50V" H 2010 6220 50  0000 L CNN
+F 2 "Capacitors_SMD:c_elec_6.3x5.3" H 2000 6300 50  0001 C CNN
+F 3 "" H 2000 6300 50  0001 C CNN
+	1    2000 6300
+	1    0    0    -1
+$EndComp
+$Comp
+L CP1_Small C36
+U 1 1 5A836099
+P 3050 6300
+F 0 "C36" H 3060 6370 50  0000 L CNN
+F 1 "22uF/50V" H 3060 6220 50  0000 L CNN
+F 2 "Capacitors_SMD:c_elec_6.3x5.3" H 3050 6300 50  0001 C CNN
+F 3 "" H 3050 6300 50  0001 C CNN
+	1    3050 6300
+	1    0    0    -1
+$EndComp
+$Comp
+L CP1_Small C37
+U 1 1 5A8361BC
+P 4050 6300
+F 0 "C37" H 4060 6370 50  0000 L CNN
+F 1 "22uF/50V" H 4060 6220 50  0000 L CNN
+F 2 "Capacitors_SMD:c_elec_6.3x5.3" H 4050 6300 50  0001 C CNN
+F 3 "" H 4050 6300 50  0001 C CNN
+	1    4050 6300
+	1    0    0    -1
+$EndComp
 $EndSCHEMATC

Commit message: ALim a grosse piste
Parts:
- removed C26, C27, C28, C29, C30: 100uF, Capacitors_Tantalum_SMD:Tantalum_Case-B_EIA-3528-21_Hand, symbol CP1_Small
- removed C35, C36, C37: 22uF/50V, Capacitors_SMD:c_elec_6.3x5.3, symbol CP1_Small
- removed P1: BATT_IN, kicad-library:BATT_SOLDERPAD, symbol CONN_01X02
- removed P2: ALIM_L1, Pin_Headers:Pin_Header_Straight_2x03, symbol CONN_02X03
- removed P5: SW_LOGIC, Socket_Strips:Socket_Strip_Straight_1x02, symbol CONN_01X02
- removed Q6: Q_PMOS_GDS, TO_SOT_Packages_SMD:SOT-428, symbol Q_PMOS_GDS
- removed R15: 10k, Resistors_SMD:R_0603_HandSoldering, symbol R_Small
- removed R17: 8k, Resistors_SMD:R_0603_HandSoldering, symbol R_Small
- removed U2: TRACO3.3, kicad-library:TRACO-TSR-1-DC-DC, symbol 7805-RESCUE-Alimentation_2017
- removed U3: TRACO5, kicad-library:TRACO-TSR-1-DC-DC, symbol 7805-RESCUE-Alimentation_2017
- removed U4: TRACO15, kicad-library:TRACO-TSR-1-DC-DC, symbol 7805-RESCUE-Alimentation_2017
- added P1: BAT1+, kicad-library:WireConnection_2.50mm, symbol CONN_01X01
- added P2: BAT1-, kicad-library:WireConnection_2.50mm, symbol CONN_01X01
- added P5: BAT2+, kicad-library:WireConnection_2.50mm, symbol CONN_01X01
- added P6: BAT2-, kicad-library:WireConnection_2.50mm, symbol CONN_01X01
- C16, C17, C18, C19: value 100uF -> 270uF; footprint Capacitors_Tantalum_SMD:Tantalum_Case-B_EIA-3528-21_Hand -> Capacitors_SMD:c_elec_6.3x7.7
Connections:
- net FBCK1: now also U1.16 (FB2); no longer U1.9 (FB1)
- net FBCK2: now also U1.9 (FB1); no longer U1.16 (FB2)
- net GND: now also P6.1 (P1); no longer P3.32 (P32)
- net VBATT: now also P3.32 (P32)
- net at C10.1, D1.2 (A): now also U1.24 (VCC2); no longer U1.1 (VCC1)
- net at C6.2, R4.2: now also U1.15 (COMP2); no longer U1.10 (COMP1)
- net at U1.2 (LO1): now also Q4.2 (G); no longer Q2.2 (G)
- net at C11.2, D1.1 (K): now also U1.27 (HB2); no longer U1.30 (HB1)
- net at U1.31 (HO1): now also Q3.2 (G); no longer Q1.2 (G)
- net at C11.1, L1.1, Q1.3 (S)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: now also U1.25 (SW2); no longer U1.32 (SW1)
- net at Q2.3 (S), R6.1: now also U1.20 (CS2); no longer U1.5 (CS1)
- net at C7.1, R5.2: now also U1.19 (RAMP2); no longer U1.6 (RAMP1)
- net at U1.7 (SS1): now also C15.1; no longer C9.1
- net at C12.2, R7.2: now also U1.10 (COMP1); no longer U1.15 (COMP2)
- net at U1.18 (SS2): now also C9.1; no longer C15.1
- net at C13.1, R10.1: now also U1.6 (RAMP1); no longer U1.19 (RAMP2)
- net at Q4.3 (S), R11.1: now also U1.5 (CS1); no longer U1.20 (CS2)
- net at U1.23 (LO2): now also Q2.2 (G); no longer Q4.2 (G)
- net at C23.1, D2.2 (A): now also U1.1 (VCC1); no longer U1.24 (VCC2)
- net at C31.2, L2.1, Q3.3 (S)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: now also U1.32 (SW1); no longer U1.25 (SW2)
- net at U1.26 (HO2): now also Q1.2 (G); no longer Q3.2 (G)
- net at C31.1, D2.1 (K): now also U1.30 (HB1); no longer U1.27 (HB2)
- net at F1.1: now also P1.1 (P1)
- new net: P2.1 (P1), P5.1 (P1)
Other:
- moved on the sheet: U1A, U1B

Commit message: Couleur
Parts:
- R11: value 3M1W -> 3m1W
- R6: value 5M1.5W -> 5m1.5W
Changed lines of the file:
@@
 P 7400 3050
 F 0 "R6" H 7430 3070 50  0000 L CNN
-F 1 "5M1.5W" H 7430 3010 50  0000 L CNN
+F 1 "5m1.5W" H 7430 3010 50  0000 L CNN
 F 2 "Resistors_SMD:R_2010_HandSoldering" H 7400 3050 50  0001 C CNN
 F 3 "" H 7400 3050 50  0001 C CNN
@@
 P 10150 3050
 F 0 "R11" H 10180 3070 50  0000 L CNN
-F 1 "3M1W" H 10180 3010 50  0000 L CNN
+F 1 "3m1W" H 10180 3010 50  0000 L CNN
 F 2 "Resistors_SMD:R_2010_HandSoldering" H 10150 3050 50  0001 C CNN
 F 3 "" H 10150 3050 50  0001 C CNN

Commit message: maj
Parts:
- R16: value 8k -> 7.15k
Changed lines of the file:
@@
 P 1350 1900
 F 0 "R16" V 1250 1850 50  0000 L CNN
-F 1 "8k" V 1350 1850 50  0000 L CNN
+F 1 "7.15k" V 1400 2000 50  0000 L CNN
 F 2 "Resistors_SMD:R_0603_HandSoldering" H 1350 1900 50  0001 C CNN
 F 3 "" H 1350 1900 50  0001 C CNN

Commit message: Alim protodual
Parts:
- removed Q1, Q2, Q3, Q4: Q_NMOS_DGS, kicad-library:TDSON8_MOSFET, symbol Q_NMOS_DGS
- added Q1, Q2, Q3, Q4: Q_NMOS_SGD, kicad-library:TDSON8_MOSFET, symbol Q_NMOS_SGD
Connections:
- net +BATT: now also Q5.2 (D), Q1.3 (D), Q3.3 (D); no longer Q5.3 (S)
- net VBATT: now also Q5.3 (S); no longer Q5.2 (D)
- net at U1.2 (LO1): now also Q4.2 (G)
- net at U1.31 (HO1): now also Q3.2 (G)
- net at C31.2, L2.1, R10.2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: now also Q3.1 (S), Q4.3 (D)
- net at R11.1, U1.5 (CS1): now also Q4.1 (S)
- net at R6.1, U1.20 (CS2): now also Q2.1 (S)
- net at U1.23 (LO2): now also Q2.2 (G)
- net at C11.1, L1.1, R5.1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: now also Q1.1 (S), Q2.3 (D)
- net at U1.26 (HO2): now also Q1.2 (G)
Changed lines of the file:
@@
-$EndComp
-$Comp
-L Q_NMOS_DGS Q1
-U 1 1 5A36E47F
-P 7300 2150
-F 0 "Q1" H 7500 2200 50  0000 L CNN
-F 1 "Q_NMOS_DGS" H 7500 2100 50  0000 L CNN
-F 2 "kicad-library:TDSON8_MOSFET" H 7500 2250 50  0001 C CNN
-F 3 "" H 7300 2150 50  0001 C CNN
-	1    7300 2150
-	1    0    0    -1
-$EndComp
-$Comp
-L Q_NMOS_DGS Q2
-U 1 1 5A36E54C
-P 7300 2650
-F 0 "Q2" H 7500 2700 50  0000 L CNN
-F 1 "Q_NMOS_DGS" H 7500 2600 50  0000 L CNN
-F 2 "kicad-library:TDSON8_MOSFET" H 7500 2750 50  0001 C CNN
-F 3 "" H 7300 2650 50  0001 C CNN
-	1    7300 2650
-	1    0    0    -1
 $EndComp
 $Comp
@@
 FBCK1
 $Comp
-L Q_NMOS_DGS Q3
-U 1 1 5A3B253A
-P 10050 2150
-F 0 "Q3" H 10250 2200 50  0000 L CNN
-F 1 "Q_NMOS_DGS" H 10250 2100 50  0000 L CNN
-F 2 "kicad-library:TDSON8_MOSFET" H 10250 2250 50  0001 C CNN
-F 3 "" H 10050 2150 50  0001 C CNN
-	1    10050 2150
-	1    0    0    -1
-$EndComp
-$Comp
-L Q_NMOS_DGS Q4
-U 1 1 5A3B2629
-P 10050 2650
-F 0 "Q4" H 10250 2700 50  0000 L CNN
-F 1 "Q_NMOS_DGS" H 10250 2600 50  0000 L CNN
-F 2 "kicad-library:TDSON8_MOSFET" H 10250 2750 50  0001 C CNN
-F 3 "" H 10050 2650 50  0001 C CNN
-	1    10050 2650
-	1    0    0    -1
-$EndComp
-$Comp
 L R_Small R11
 U 1 1 5A3B2782
@@
 F 3 "" H 1850 1750 50  0001 C CNN
 	1    1850 1750
-	1    0    0    -1
+	1    0    0    1
 $EndComp
 Wire Wire Line
@@
 Wire Wire Line
 	8650 500  8650 1000
+$Comp
+L Q_NMOS_SGD Q1
+U 1 1 5AB7B835
+P 7300 2150
+F 0 "Q1" H 7500 2200 50  0000 L CNN
+F 1 "Q_NMOS_SGD" H 7500 2100 50  0000 L CNN
+F 2 "kicad-library:TDSON8_MOSFET" H 7500 2250 50  0001 C CNN
+F 3 "" H 7300 2150 50  0001 C CNN
+	1    7300 2150
+	1    0    0    -1
+$EndComp
+$Comp
+L Q_NMOS_SGD Q2
+U 1 1 5AB7BC11
+P 7300 2650
+F 0 "Q2" H 7500 2700 50  0000 L CNN
+F 1 "Q_NMOS_SGD" H 7500 2600 50  0000 L CNN
+F 2 "kicad-library:TDSON8_MOSFET" H 7500 2750 50  0001 C CNN
+F 3 "" H 7300 2650 50  0001 C CNN
+	1    7300 2650
+	1    0    0    -1
+$EndComp
+$Comp
+L Q_NMOS_SGD Q3
+U 1 1 5AB7BCF4
+P 10050 2150
+F 0 "Q3" H 10250 2200 50  0000 L CNN
+F 1 "Q_NMOS_SGD" H 10250 2100 50  0000 L CNN
+F 2 "kicad-library:TDSON8_MOSFET" H 10250 2250 50  0001 C CNN
+F 3 "" H 10050 2150 50  0001 C CNN
+	1    10050 2150
+	1    0    0    -1
+$EndComp
+$Comp
+L Q_NMOS_SGD Q4
+U 1 1 5AB7BDF2
+P 10050 2650
+F 0 "Q4" H 10250 2700 50  0000 L CNN
+F 1 "Q_NMOS_SGD" H 10250 2600 50  0000 L CNN
+F 2 "kicad-library:TDSON8_MOSFET" H 10250 2750 50  0001 C CNN
+F 3 "" H 10050 2650 50  0001 C CNN
+	1    10050 2650
+	1    0    0    -1
+$EndComp
 $EndSCHEMATC
