File: alim/protodual.kicad_pcb (KiCad board)
At the start: 2 copper layers, 72 parts, among them P1 BATT_IN, P2 ALIM_L1, P3 ALIM_PW1, P4 ARU, P5 SW_LOGIC, Q1 Q_NMOS_DGS, Q2 Q_NMOS_DGS, Q3 Q_NMOS_DGS, Q4 Q_NMOS_DGS, Q5 Q_PMOS_GDS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

Commit message: alim
Parts:
- C2, C3: moved to B.Cu
- moved C3 72.3 mm to (175.3, 105.4)
- moved C2 41.7 mm to (130.8, 105.9)
Routing:
- net GND: track 313.9 -> 620.0 mm, vias 2 -> 4
- net +BATT: track 169.2 -> 182.4 mm
- net VOUT2: track 98.0 -> 110.7 mm
- net VOUT1: track 126.6 -> 139.3 mm
- net Net-(C31-Pad2): track 50.1 -> 61.9 mm
- net Net-(C11-Pad1): track 35.1 -> 41.5 mm
- net VBATT: track 62.2 -> 59.9 mm
Other:
- board outline added: 99.6 x 87.4 mm

Commit message: Alim finale?
Parts:
- added R16: 1k, Resistors_SMD:R_0603_HandSoldering, F.Cu at (98.6, 118.4)
- added R17: 1k, Resistors_SMD:R_0603_HandSoldering, F.Cu at (109.2, 118.4)
- R14, R15: value 10k -> 20k
- moved P4 1.27 mm to (103.4, 119.9)
- moved P5 1.02 mm to (113.8, 119.9)
Connections:
- P4 pad 1: +BATT -> GND
- P5 pad 1: Net-(C35-Pad1) -> GND
- Q5 pad 1: Net-(P4-Pad2) -> Net-(Q5-Pad1)
- Q6 pad 1: Net-(P5-Pad2) -> Net-(Q6-Pad1)
- R14 pad 2: Net-(P4-Pad2) -> Net-(Q5-Pad1)
- R15 pad 2: Net-(P5-Pad2) -> Net-(Q6-Pad1)
Routing:
- net GND: track 620.0 -> 651.3 mm, vias 4 -> 5
- net Net-(Q5-Pad1): track 0.00 -> 6.38 mm
- net Net-(Q6-Pad1): track 0.00 -> 5.36 mm
- net Net-(P5-Pad2): track 6.31 -> 2.21 mm
- net +BATT: track 182.4 -> 178.7 mm
- net Net-(C35-Pad1): track 131.4 -> 127.7 mm
- net Net-(P4-Pad2): track 6.82 -> 3.37 mm

Commit message: Alim
Parts:
- removed C36, C37: 22uF/50V, Capacitors_SMD:C_1206_HandSoldering
- C35: footprint Capacitors_SMD:C_1206_HandSoldering -> Capacitors_SMD:c_elec_6.3x5.3
- D1, D2: footprint Diodes_SMD:SMC_Handsoldering -> Diodes_SMD:D_0805
- R14, R15: value 20k -> 10k
- R16, R17: value 1k -> 8k
- moved D1 7.11 mm to (143.8, 106.7)
- moved D2 6.23 mm to (159.8, 105.7)
- moved C35 3.70 mm to (181.4, 98.6)
Routing:
- net Net-(C10-Pad1): track 20.5 -> 8.78 mm
- net GND: track 651.3 -> 659.1 mm
- net Net-(C11-Pad2): track 13.4 -> 7.54 mm
- net Net-(C23-Pad1): track 17.9 -> 12.3 mm
- net Net-(C31-Pad1): track 15.0 -> 11.8 mm

Commit message: ALim a grosse piste
Parts:
- removed C26, C27, C28, C29, C30: 100uF, Capacitors_Tantalum_SMD:Tantalum_Case-B_EIA-3528-21_Hand
- removed C35: 22uF/50V, Capacitors_SMD:c_elec_6.3x5.3
- removed Q6: Q_PMOS_GDS, TO_SOT_Packages_SMD:SOT-428
- removed R15: 10k, Resistors_SMD:R_0603_HandSoldering
- removed R17: 8k, Resistors_SMD:R_0603_HandSoldering
- removed U2: TRACO3.3, kicad-library:TRACO-TSR-1-DC-DC
- removed U3: TRACO5, kicad-library:TRACO-TSR-1-DC-DC
- removed U4: TRACO15, kicad-library:TRACO-TSR-1-DC-DC
- added P6: BAT2-, kicad-library:WireConnection_2.50mm, F.Cu at (99.3, 132.5)
- added REF**: MountingHole_2.7mm_M2.5_ISO14580, Mounting_Holes:MountingHole_2.7mm_M2.5_ISO14580, F.Cu at (186.0, 101.0)
- added REF**: MountingHole_2.7mm_M2.5_ISO14580, Mounting_Holes:MountingHole_2.7mm_M2.5_ISO14580, F.Cu at (186.0, 138.0)
- added REF**: MountingHole_2.7mm_M2.5_ISO14580, Mounting_Holes:MountingHole_2.7mm_M2.5_ISO14580, F.Cu at (92.0, 138.0)
- C15, C5, C9, R1, R12, R13, R2, R8, R9: moved to B.Cu
- C16, C17, C18, C19: value 100uF -> 270uF; footprint Capacitors_Tantalum_SMD:Tantalum_Case-B_EIA-3528-21_Hand -> Capacitors_SMD:c_elec_6.3x7.7; moved to F.Cu
- C2, C21, C24, C3: moved to F.Cu
- P1: value BATT_IN -> BAT1+; footprint kicad-library:BATT_SOLDERPAD -> kicad-library:WireConnection_2.50mm
- P2: value ALIM_L1 -> BAT1-; footprint Pin_Headers:Pin_Header_Straight_2x03 -> kicad-library:WireConnection_2.50mm
- P5: value SW_LOGIC -> BAT2+; footprint Socket_Strips:Socket_Strip_Straight_1x02 -> kicad-library:WireConnection_2.50mm
- moved P2 101.6 mm to (99.3, 120.0), turned to 180 degrees
- moved C18 76.6 mm to (183.7, 107.2), turned to 0 degrees
- moved C17 75.5 mm to (183.7, 114.5), turned to 0 degrees
- moved C16 74.0 mm to (183.7, 129.0), turned to 0 degrees
- moved C33 74.0 mm to (108.5, 119.8), turned to 180 degrees
- moved C34 73.9 mm to (108.5, 134.2), turned to 180 degrees
- moved C32 66.2 mm to (108.5, 127.0), turned to 180 degrees
- moved R6 55.3 mm to (176.5, 105.7), turned to 90 degrees
- moved C19 53.8 mm to (183.7, 121.8)
- moved C24 53.1 mm to (163.2, 132.1), turned to 90 degrees
- moved C21 52.2 mm to (179.9, 138.2)
- moved C22 50.1 mm to (179.8, 134.5)
- moved Q2 49.3 mm to (172.8, 113.4), turned to 0 degrees
- moved C20 45.4 mm to (179.9, 134.5)
- moved R11 44.9 mm to (138.6, 124.5), turned to 180 degrees
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Connections:
- P1 pad 1: GND -> Net-(F1-Pad1)
- P2 pad 1: VL33 -> Net-(P2-Pad1)
- P3 pad 32: GND -> VBATT
- P5 pad 1: GND -> Net-(P2-Pad1)
- U1 pad 1: Net-(C10-Pad1) -> Net-(C23-Pad1)
- U1 pad 10: Net-(C6-Pad2) -> Net-(C12-Pad2)
- U1 pad 15: Net-(C12-Pad2) -> Net-(C6-Pad2)
- U1 pad 16: FBCK2 -> FBCK1
- U1 pad 18: Net-(C15-Pad1) -> Net-(C9-Pad1)
- U1 pad 19: Net-(C13-Pad1) -> Net-(C7-Pad1)
- U1 pad 2: Net-(Q2-Pad2) -> Net-(Q4-Pad2)
- U1 pad 20: Net-(Q4-Pad3) -> Net-(Q2-Pad3)
- U1 pad 23: Net-(Q4-Pad2) -> Net-(Q2-Pad2)
- U1 pad 24: Net-(C23-Pad1) -> Net-(C10-Pad1)
- U1 pad 25: Net-(C31-Pad2) -> Net-(C11-Pad1)
- U1 pad 26: Net-(Q3-Pad2) -> Net-(Q1-Pad2)
- U1 pad 27: Net-(C31-Pad1) -> Net-(C11-Pad2)
- U1 pad 30: Net-(C11-Pad2) -> Net-(C31-Pad1)
- U1 pad 31: Net-(Q1-Pad2) -> Net-(Q3-Pad2)
- U1 pad 32: Net-(C11-Pad1) -> Net-(C31-Pad2)
- U1 pad 5: Net-(Q2-Pad3) -> Net-(Q4-Pad3)
- U1 pad 6: Net-(C7-Pad1) -> Net-(C13-Pad1)
- U1 pad 7: Net-(C9-Pad1) -> Net-(C15-Pad1)
- U1 pad 9: FBCK1 -> FBCK2
Routing:
- net GND: track 659.1 -> 52.2 mm
- net Net-(C35-Pad1): track 127.7 -> 0.00 mm, vias 2 -> 0
- net VOUT1: track 139.3 -> 15.8 mm
- net VOUT2: track 110.7 -> 28.2 mm, vias 0 -> 3
- net +BATT: track 178.7 -> 97.8 mm, vias 4 -> 1
- net VL15: track 54.8 -> 0.00 mm
- net Net-(C31-Pad2): track 61.9 -> 16.7 mm, vias 0 -> 2
- net VL33: track 33.6 -> 0.00 mm
- net Net-(Q4-Pad3): track 37.4 -> 11.2 mm
- net Net-(C11-Pad1): track 41.5 -> 19.8 mm, vias 0 -> 2
- net Net-(Q4-Pad2): track 29.1 -> 14.6 mm
- net VL5: track 14.0 -> 0.00 mm
- net Net-(Q2-Pad3): track 36.0 -> 24.1 mm
- net Net-(Q2-Pad2): track 26.3 -> 15.8 mm
- net Net-(C13-Pad1): track 12.1 -> 4.05 mm, vias 2 -> 0
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- added copper zone on F.Cu, net +BATT
- added copper zone on B.Cu, net GND
- added copper zone on F.Cu, net Net-(C11-Pad1)
- added copper zone on F.Cu, net Net-(C31-Pad2)
- added copper zone on F.Cu, net Net-(P2-Pad1)
- added copper zone on F.Cu, net Net-(Q2-Pad3)
- added copper zone on F.Cu, net Net-(Q4-Pad3)
- added copper zone on F.Cu, net VOUT1
- added copper zone on F.Cu, net VOUT2
Other:
- board size 99.6 x 87.4 mm -> 100 x 43 mm
- net class Power: trace_width 2 -> 4; via_dia 1 -> 3; via_drill 0.4 -> 2
- net class VBatt added: clearance 0.8, trace_width 1, via_dia 0.8, via_drill 0.5

Commit message: Alim
Parts:
- renumbered REF** to ?
Routing:
- net Net-(P2-Pad1): track 0.00 -> 22.7 mm
- net GND: track 52.2 -> 64.3 mm, vias 5 -> 4
- net Net-(F1-Pad1): track 15.6 -> 13.3 mm
- net (no net): vias 0 -> 1
- removed copper zone on F.Cu, net Net-(P2-Pad1)
Other:
- net class VBatt: trace_width 1 -> 5; via_dia 0.8 -> 3
- board text added: "+32V"
- board text added: "GND"

Commit message: maj
Routing:
- net VOUT1: track 15.8 -> 23.7 mm, vias 1 -> 3
Other:
- outline, holes or cut-outs redrawn
- net class Power: trace_width 4 -> 3
Changed lines of the file:
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@@
   (general
     (links 194)
-    (no_connects 9)
+    (no_connects 7)
     (area 88.924999 97.924999 189.075001 141.075001)
     (thickness 1.6)
-    (drawings 6)
-    (tracks 288)
+    (drawings 10)
+    (tracks 292)
     (zones 0)
     (modules 64)
@@
   )
   (page A4)
+  (title_block
+    (title "La double Alimentation")
+    (company Aigris)
+    (comment 1 VOUT1=6V)
+    (comment 2 VOUT2=12V)
+  )
   (layers
     (0 F.Cu signal)
     (31 B.Cu signal)
-    (32 B.Adhes user hide)
+    (32 B.Adhes user)
     (33 F.Adhes user)
-    (34 B.Paste user hide)
+    (34 B.Paste user)
     (35 F.Paste user)
-    (36 B.SilkS user hide)
+    (36 B.SilkS user)
     (37 F.SilkS user)
-    (38 B.Mask user hide)
+    (38 B.Mask user)
     (39 F.Mask user)
     (40 Dwgs.User user)
@@
     (44 Edge.Cuts user)
     (45 Margin user)
-    (46 B.CrtYd user hide)
+    (46 B.CrtYd user)
     (47 F.CrtYd user)
-    (48 B.Fab user hide)
+    (48 B.Fab user)
     (49 F.Fab user)
   )
@@
     (visible_elements FFFEFFFF)
     (pcbplotparams
-      (layerselection 0x00030_80000001)
+      (layerselection 0x010f0_80000001)
       (usegerberextensions false)
       (excludeedgelayer true)
@@
       (outputformat 1)
       (mirror false)
-      (drillshape 1)
+      (drillshape 0)
       (scaleselection 1)
-      (outputdirectory ""))
+      (outputdirectory gerber/))
   )
   (net 0 "")
@@
     (add_net "Net-(U1-Pad8)")
     (add_net VBATT)
-    (add_net VOUT1)
     (add_net VOUT2)
   )
@@
   (net_class Power ""
     (clearance 0.2)
-    (trace_width 4)
+    (trace_width 3)
     (via_dia 3)
     (via_drill 2)
     (uvia_dia 0.3)
     (uvia_drill 0.1)
+    (add_net VOUT1)
   )
   (net_class VBatt ""
@@
     (tags "capacitor 0805")
     (attr smd)
-    (fp_text reference C9 (at 0 2.1) (layer B.SilkS)
+    (fp_text reference C9 (at 3 0) (layer B.SilkS)
       (effects (font (size 1 1) (thickness 0.15)) (justify mirror))
     )
@@
     (tags "capacitor tantalum smd")
     (attr smd)
-    (fp_text reference C22 (at 0 3.15) (layer B.SilkS)
+    (fp_text reference C22 (at -4.85 0.25 90) (layer B.SilkS)
       (effects (font (size 1 1) (thickness 0.15)) (justify mirror))
     )
@@
     (tags "capacitor tantalum smd")
     (attr smd)
-    (fp_text reference C25 (at 0 3.15) (layer B.SilkS)
+    (fp_text reference C25 (at -4.9 0 90) (layer B.SilkS)
       (effects (font (size 1 1) (thickness 0.15)) (justify mirror))
     )
@@
     (tags "tdson ")
     (attr smd)
-    (fp_text reference Q1 (at -0.02 -3.68 270) (layer F.SilkS)
+    (fp_text reference Q1 (at -1.75 3.25 270) (layer F.SilkS)
       (effects (font (size 1 1) (thickness 0.15)))
     )
@@
     (tags "resistor 0603")
     (attr smd)
-    (fp_text reference R8 (at 0 1.9 180) (layer B.SilkS)
+    (fp_text reference R8 (at -3.1 0 180) (layer B.SilkS)
       (effects (font (size 1 1) (thickness 0.15)) (justify mirror))
     )
@@
     (tags "resistor 0603")
     (attr smd)
-    (fp_text reference R10 (at 2.6 -0.75 270) (layer F.SilkS)
+    (fp_text reference R10 (at 1.4 -1.5 360) (layer F.SilkS)
       (effects (font (size 1 1) (thickness 0.15)))
     )
@@
     (tags "resistor 0603")
     (attr smd)
-    (fp_text reference R12 (at 0 1.9) (layer B.SilkS)
+    (fp_text reference R12 (at 0 -1.25) (layer B.SilkS)
       (effects (font (size 1 1) (thickness 0.15)) (justify mirror))
     )
@@
     (tags "resistor 0603")
     (attr smd)
-    (fp_text reference R13 (at 0 1.9 180) (layer B.SilkS)
+    (fp_text reference R13 (at 0 -1.25 180) (layer B.SilkS)
       (effects (font (size 1 1) (thickness 0.15)) (justify mirror))
     )
@@
     )
   )
+  (gr_arc (start 187 100) (end 187 98) (angle 90) (layer Edge.Cuts) (width 0.15))
+  (gr_arc (start 187 139) (end 189 139) (angle 90) (layer Edge.Cuts) (width 0.15))
+  (gr_arc (start 91 139) (end 91 141) (angle 90) (layer Edge.Cuts) (width 0.15))
+  (gr_arc (start 91 100) (end 89 100) (angle 90) (layer Edge.Cuts) (width 0.15))
   (gr_text +32V (at 99.25 107.25) (layer F.SilkS)
     (effects (font (size 1.5 1.5) (thickness 0.3)))
@@
     (effects (font (size 1.5 1.5) (thickness 0.3)))
   )
-  (gr_line (start 89 98) (end 89 141) (angle 90) (layer Edge.Cuts) (width 0.15))
-  (gr_line (start 189 98) (end 89 98) (angle 90) (layer Edge.Cuts) (width 0.15))
-  (gr_line (start 189 141) (end 189 98) (angle 90) (layer Edge.Cuts) (width 0.15))
-  (gr_line (start 89 141) (end 189 141) (angle 90) (layer Edge.Cuts) (width 0.15))
+  (gr_line (start 89 99.25) (end 89 139) (angle 90) (layer Edge.Cuts) (width 0.15))
+  (gr_line (start 187 98) (end 91 98) (angle 90) (layer Edge.Cuts) (width 0.15))
+  (gr_line (start 189 139) (end 189 100) (angle 90) (layer Edge.Cuts) (width 0.15))
+  (gr_line (start 91 141) (end 187 141) (angle 90) (layer Edge.Cuts) (width 0.15))
   (via (at 161 111.5) (size 0.6) (drill 0.4) (layers F.Cu B.Cu) (net 0))
   (segment (start 135.2 99.5) (end 135.425 99.5) (width 0.25) (layer F.Cu) (net 1))
@@
   (via (at 154 109.75) (size 0.6) (drill 0.4) (layers F.Cu B.Cu) (net 26))
   (segment (start 153.5 121.8) (end 153.5 117) (width 0.25) (layer F.Cu) (net 27))
+  (segment (start 177.7 134.5) (end 173.75 134.5) (width 3) (layer B.Cu) (net 31))
+  (via (at 173.75 134.5) (size 3) (drill 2) (layers F.Cu B.Cu) (net 31))
+  (segment (start 177.75 138.5) (end 173.75 138.5) (width 3) (layer B.Cu) (net 31))
+  (via (at 173.75 138.5) (size 3) (drill 2) (layers F.Cu B.Cu) (net 31))
   (segment (start 163.5 120.25) (end 161.25 120.25) (width 0.25) (layer B.Cu) (net 31))
   (segment (start 171.75 129.5) (end 171.75 127) (width 0.25) (layer F.Cu) (net 31))

Commit message: Alim protodual
Parts:
- Q1, Q2, Q3, Q4: value Q_NMOS_DGS -> Q_NMOS_SGD
- R11: value 3M1W -> 3m1W
- R16: value 8k -> 7.15k
- R6: value 5M1.5W -> 5m1.5W
- moved Q2 2.09 mm to (174.8, 113.5), turned to 270 degrees
- moved Q1 2.03 mm to (168.2, 112.8), turned to 180 degrees
- moved R6 0.84 mm to (176.2, 104.8)
- moved C15 0.79 mm to (147.2, 116.5)
- moved L1 0.75 mm to (171.8, 125.0)
- moved C13 0.40 mm to (147.1, 115.5)
- moved Q4 0.27 mm to (141.0, 118.2), turned to 90 degrees
- moved R11 0.25 mm to (138.6, 124.8)
- moved Q5 0.25 mm to (119.8, 105.3), turned to 180 degrees
- moved Q3 0.09 mm to (141.0, 110.5), turned to 90 degrees
Connections:
- Q1 pad 1: +BATT -> Net-(C11-Pad1)
- Q1 pad 3: Net-(C11-Pad1) -> +BATT
- Q2 pad 1: Net-(C11-Pad1) -> Net-(Q2-Pad1)
- Q2 pad 3: Net-(Q2-Pad3) -> Net-(C11-Pad1)
- Q3 pad 1: +BATT -> Net-(C31-Pad2)
- Q3 pad 3: Net-(C31-Pad2) -> +BATT
- Q4 pad 1: Net-(C31-Pad2) -> Net-(Q4-Pad1)
- Q4 pad 3: Net-(Q4-Pad3) -> Net-(C31-Pad2)
- Q5 pad 2: VBATT -> +BATT
- Q5 pad 3: +BATT -> VBATT
- R11 pad 1: Net-(Q4-Pad3) -> Net-(Q4-Pad1)
- R6 pad 1: Net-(Q2-Pad3) -> Net-(Q2-Pad1)
- U1 pad 20: Net-(Q2-Pad3) -> Net-(Q2-Pad1)
- U1 pad 5: Net-(Q4-Pad3) -> Net-(Q4-Pad1)
Routing:
- net GND: track 64.3 -> 233.5 mm, vias 4 -> 8
- net Net-(Q2-Pad3): track 24.1 -> 0.00 mm, vias 2 -> 0
- net Net-(Q4-Pad1): track 0.00 -> 23.7 mm, vias 0 -> 2
- net Net-(Q2-Pad1): track 0.00 -> 20.3 mm, vias 0 -> 2
- net Net-(Q4-Pad3): track 11.2 -> 0.00 mm, vias 2 -> 0
- net Net-(Q5-Pad1): track 4.77 -> 14.8 mm
- net Net-(Q1-Pad2): track 11.7 -> 19.7 mm
- net VBATT: track 67.3 -> 60.5 mm
- net Net-(C11-Pad1): track 19.8 -> 26.1 mm
- net Net-(Q3-Pad2): track 17.8 -> 13.5 mm, vias 2 -> 3
- net Net-(Q2-Pad2): track 15.8 -> 19.0 mm
- net Net-(C5-Pad1): track 0.00 -> 2.43 mm, vias 0 -> 1
- net Net-(C31-Pad2): track 16.7 -> 18.7 mm
- net +BATT: track 97.8 -> 96.8 mm
- net (no net): vias 1 -> 0
- added copper zone on F.Cu, net Net-(Q2-Pad1)
- added copper zone on F.Cu, net Net-(Q4-Pad1)
- removed copper zone on F.Cu, net Net-(Q2-Pad3)
- removed copper zone on F.Cu, net Net-(Q4-Pad3)

Commit message: alims
Routing:
- net GND: track 233.5 -> 236.6 mm, vias 8 -> 10
- net Net-(F1-Pad1): track 13.3 -> 15.6 mm
- added copper zone on F.Cu, net VBATT
Other:
- net class Default: clearance 0.2 -> 0.15
- net class VBatt: clearance 0.8 -> 0.2
- rule trace_clearance: 0.2 -> 0.15
Changed lines of the file:
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@@
   (general
     (links 194)
-    (no_connects 5)
-    (area 88.924999 97.924999 189.075001 141.075001)
+    (no_connects 0)
+    (area 77.128572 96.025 200.871429 143.075)
     (thickness 1.6)
     (drawings 10)
-    (tracks 354)
+    (tracks 359)
     (zones 0)
     (modules 64)
@@
   (setup
     (last_trace_width 0.25)
-    (trace_clearance 0.2)
+    (trace_clearance 0.15)
     (zone_clearance 0.508)
     (zone_45_only no)
@@
   (net 37 "Net-(Q4-Pad1)")
   (net_class Default "This is the default net class."
-    (clearance 0.2)
+    (clearance 0.15)
     (trace_width 0.25)
     (via_dia 0.6)
@@
   )
   (net_class VBatt ""
-    (clearance 0.8)
+    (clearance 0.2)
     (trace_width 5)
     (via_dia 3)
@@
   (segment (start 126.5 106.75) (end 126.5 127.816399) (width 4) (layer F.Cu) (net 1))
   (segment (start 126.5 127.816399) (end 126.62 127.936399) (width 4) (layer F.Cu) (net 1))
+  (segment (start 145.25 121.25) (end 145.25 122.5) (width 0.25) (layer B.Cu) (net 2))
+  (segment (start 145.5 118.5) (end 145.5 121) (width 0.25) (layer F.Cu) (net 2))
+  (segment (start 145.5 121) (end 145.25 121.25) (width 0.25) (layer F.Cu) (net 2))
+  (via (at 145.25 121.25) (size 0.6) (drill 0.4) (layers F.Cu B.Cu) (net 2))
+  (segment (start 146 116.5) (end 146 118) (width 0.25) (layer B.Cu) (net 2))
+  (via (at 145.5 118.5) (size 0.6) (drill 0.4) (layers F.Cu B.Cu) (net 2))
+  (segment (start 146 118) (end 145.5 118.5) (width 0.25) (layer B.Cu) (net 2))
   (segment (start 106.5 110.75) (end 106.5 107.5) (width 0.25) (layer B.Cu) (net 2))
   (segment (start 110.499999 100.500001) (end 106.5 104.5) (width 0.25) (layer B.Cu) (net 2))
@@
   (segment (start 179.5 102.5) (end 180.5 101.5) (width 4) (layer F.Cu) (net 2))
   (via (at 180.5 101.5) (size 3) (drill 2) (layers F.Cu B.Cu) (net 2))
-  (segment (start 182.05 134.5) (end 185.25 134.5) (width 4) (layer F.Cu) (net 2))
   (segment (start 185.25 134.5) (end 186 133.75) (width 4) (layer F.Cu) (net 2))
   (via (at 186 133.75) (size 3) (drill 2) (layers F.Cu B.Cu) (net 2))
@@
   (segment (start 152 117) (end 152 117.75) (width 0.25) (layer F.Cu) (net 13))
   (segment (start 152 117.75) (end 151 118.75) (width 0.25) (layer F.Cu) (net 13))
-  (segment (start 148 115.5) (end 149.472998 115.5) (width 0.25) (layer F.Cu) (net 14))
-  (segment (start 149.472998 115.5) (end 149.497999 115.474999) (width 0.25) (layer F.Cu) (net 14))
-  (segment (start 149.497999 115.474999) (end 150.599999 115.474999) (width 0.25) (layer F.Cu) (net 14))
-  (segment (start 150.599999 115.474999) (end 150.599999 115.40001) (width 0.25) (layer F.Cu) (net 14))
+  (segment (start 150.85 115.35) (end 148.15 115.35) (width 0.25) (layer F.Cu) (net 14))
+  (segment (start 148.15 115.35) (end 148 115.5) (width 0.25) (layer F.Cu) (net 14))
   (segment (start 148.5 117) (end 148.5 115.6) (width 0.25) (layer F.Cu) (net 14))
   (segment (start 148.5 115.6) (end 148.4 115.5) (width 0.25) (layer F.Cu) (net 14))
@@
   (segment (start 157.1 128.46) (end 156.87413 128.46) (width 1) (layer B.Cu) (net 31))
   (segment (start 156.87413 128.46) (end 154.91413 126.5) (width 1) (layer B.Cu) (net 31))
+  (segment (start 91.4 103.4) (end 93 105) (width 0.25) (layer F.Cu) (net 32))
   (segment (start 93 112) (end 93 105) (width 7) (layer F.Cu) (net 32))
   (segment (start 99.35 112) (end 93 112) (width 7) (layer F.Cu) (net 32))
@@
     (polygon
       (pts
-        (xy 140.5 125.75) (xy 138.75 124) (xy 138.75 121.5) (xy 138.75 120.25) (xy 142 120.25)
-        (xy 142 122.25) (xy 143 123.25) (xy 143 125.75)
+        (xy 140.6 125.8) (xy 138.6 123.8) (xy 138.6 121.6) (xy 138.6 120.6) (xy 142 120.6)
+        (xy 142 122.25) (xy 143 123.25) (xy 143 125.8)
       )
     )
@@
     (polygon
       (pts
-        (xy 142.25 114.5) (xy 142.25 112.75) (xy 138.5 112.75) (xy 134.75 112.75) (xy 132.25 112.75)
-        (xy 129.75 115.25) (xy 129.75 122) (xy 134.25 122) (xy 136.25 120) (xy 143.25 120)
-        (xy 143.25 114.5)
+        (xy 142 114.6) (xy 142 112.8) (xy 138.4 112.8) (xy 134.8 112.8) (xy 132.2 112.8)
+        (xy 129.75 115.25) (xy 129.75 122) (xy 134.25 122) (xy 136.25 120) (xy 143.2 120)
+        (xy 143.2 114.6)
       )
     )
@@
       (pts
         (xy 123.75 122) (xy 123.75 117) (xy 121.75 115) (xy 115.5 115) (xy 112.75 115)
-        (xy 109 118.75) (xy 109 140.5) (xy 109 141) (xy 134.75 141) (xy 134.75 130)
-        (xy 117.5 130) (xy 117.5 126) (xy 121.25 122.25) (xy 121.5 122)
+        (xy 109 118.75) (xy 109 140.5) (xy 109 141) (xy 134.8 141) (xy 134.8 130.2)
+        (xy 117.6 130.2) (xy 117.6 126) (xy 121.4 122.2) (xy 121.6 122)
       )
     )
@@
     (polygon
       (pts
-        (xy 136.25 130) (xy 136.25 141) (xy 179.75 141) (xy 179.75 132.75) (xy 181.5 131)
+        (xy 136.2 130.2) (xy 136.2 141) (xy 179.6 141) (xy 179.6 132.8) (xy 181.4 131)
         (xy 182.25 131) (xy 183.25 130) (xy 183.25 106.25) (xy 179 106.25) (xy 179 120.75)
         (xy 174.75 125) (xy 170 125) (xy 167.5 127.5) (xy 167.5 132.5) (xy 153 132.5)
-        (xy 153 130)
+        (xy 153 130.2)
       )
     )
@@
     (polygon
       (pts
-        (xy 145 105) (xy 158.75 105) (xy 163.25 109.5) (xy 163.25 120.75) (xy 164.75 122.25)
-        (xy 164.75 132) (xy 153.75 132) (xy 153.75 129.5) (xy 131 129.5) (xy 131 127)
+        (xy 145 105) (xy 158.6 105) (xy 163.2 109.6) (xy 163.2 120.6) (xy 164.8 122.2)
+        (xy 164.8 131.8) (xy 153.8 131.8) (xy 153.8 129.4) (xy 131 129.4) (xy 131 127)
         (xy 132.25 127) (xy 134.25 125) (xy 136.75 125) (xy 138.75 127) (xy 145 127)
       )
@@
     (polygon
       (pts
-        (xy 174.75 106.5) (xy 174.75 108.75) (xy 173.75 109.75) (xy 173.75 111) (xy 174 111.25)
-        (xy 177.25 111.25) (xy 178 110.5) (xy 178 106.5)
+        (xy 174.8 106.6) (xy 174.8 108.8) (xy 173.8 109.8) (xy 173.8 111) (xy 174 111.2)
+        (xy 177.2 111.2) (xy 178 110.4) (xy 178 106.6)
       )
     )
@@
     (polygon
       (pts
-        (xy 124 98) (xy 124 103.5) (xy 131.25 103.5) (xy 134 100.75) (xy 134 98)
+        (xy 124 98) (xy 124 103.4) (xy 131.2 103.4) (xy 133.8 100.8) (xy 133.8 98)
       )
     )
@@
       )
     )
+  )
+  (zone (net 31) (net_name VBATT) (layer F.Cu) (hatch edge 0.508)
+    (connect_pads thru_hole_only (clearance 0.508))
+    (min_thickness 0.254)
+    (fill yes (arc_segments 16) (thermal_gap 0.508) (thermal_bridge_width 2))
+    (polygon
+      (pts
+        (xy 117.75 99) (xy 113 99) (xy 110.25 101.75) (xy 110.25 106) (xy 114.25 106)
+        (xy 114.25 105.5) (xy 116 103.75) (xy 118.25 103.75) (xy 119.25 102.75) (xy 119.25 99.75)
+        (xy 118.5 99)
+      )
+    )
