File: couleur/couleur.kicad_pcb (KiCad board)
At the start: 2 copper layers, 13.7 x 33.5 mm, 12 parts, among them P1 CONN_02X03, P2 Mounting, U1 S4282-51

Commit message: Couleur
Parts:
- removed R5: 600, Resistors_SMD:R_0603_HandSoldering
- removed R6: 122, Resistors_SMD:R_0603_HandSoldering
- removed R7: 131, Resistors_SMD:R_0603_HandSoldering
- added C2: C_Small, Capacitors_SMD:C_0603_HandSoldering, F.Cu at (182.3, 95.2)
- added C3: C_Small, Capacitors_SMD:C_0603_HandSoldering, F.Cu at (182.3, 100.0)
- added C4: C_Small, Capacitors_SMD:C_0603_HandSoldering, F.Cu at (182.3, 98.0)
Routing:
- net GND: track 12.5 -> 28.5 mm
- net +5VL: track 30.5 -> 16.7 mm
- net Net-(C2-Pad1): track 16.2 -> 16.9 mm
